File: Wearable Sound Alert System.kicad_sch (KiCad schematic)
At the start: 17 parts, among them M1 Motor_DC, U1 STM32F429ZITx, U2 TPS63030DSK, U3 MAX17261xxTD, U4 LCD-016N002L, U5 LM324

Commit message: Uploading current PCB schematics
1. split the mic-motor pairs off of main board
2. main board has footprints assigned, PCB is started, but no layout work has been done
3. Uploaded downloaded footprints used, I can upload the symbols later
Parts:
- removed C1: 4.7u, symbol Device:C
- removed C2: 0.1u, symbol Device:C
- removed M1: Motor_DC, symbol Motor:Motor_DC
- removed MK1: Microphone, symbol Device:Microphone
- removed R1, R5: 330, symbol Device:R_US
- removed R3: 680, symbol Device:R_US
- removed R4, R6: 390, symbol Device:R_US
- removed R7: 780, symbol Device:R_US
- removed RL: 2.2k, symbol Device:R_US
- removed U1: STM32F429ZITx, Package_QFP:LQFP-144_20x20mm_P0.5mm, symbol MCU_ST_STM32F4:STM32F429ZITx
- removed U2: TPS63030DSK, Package_SON:WSON-10-1EP_2.5x2.5mm_P0.5mm_EP1.2x2mm, symbol Regulator_Switching:TPS63030DSK
- removed U3: MAX17261xxTD, Package_DFN_QFN:TDFN-14-1EP_3x3mm_P0.4mm_EP1.78x2.35mm, symbol Battery_Management:MAX17261xxTD
- removed U4: LCD-016N002L, Display:LCD-016N002L, symbol Display_Character:LCD-016N002L
- removed U5: LM324, symbol Amplifier_Operational:LM324
- added C23, C24: 2.2u, Capacitor_SMD:C_0805_2012Metric_Pad1.18x1.45mm_HandSolder, symbol Device:C
- added C25, C27, C28, C29, C30, C31, C32, C33, C34, C35, C36, C37, C38, C39, C40, C42, C43, C44, C45, C46, C47, C48, CvinA1, CvinA2: 100n, Capacitor_SMD:C_0805_2012Metric_Pad1.18x1.45mm_HandSolder, symbol Device:C
- added C26, C49, C6, C7: 1u, Capacitor_SMD:C_0805_2012Metric_Pad1.18x1.45mm_HandSolder, symbol Device:C
- added C4, C50: 0.1u, Capacitor_SMD:C_0805_2012Metric_Pad1.18x1.45mm_HandSolder, symbol Device:C
- added C41: 4.7u, Capacitor_SMD:C_0805_2012Metric_Pad1.18x1.45mm_HandSolder, symbol Device:C
- added C5: 0.47p, Capacitor_SMD:C_0805_2012Metric_Pad1.18x1.45mm_HandSolder, symbol Device:C
- added Cin1, Cin3, Cout1, Cout2, Cout3, Cout4, Cout5, Cout6: 10u, Capacitor_SMD:C_0805_2012Metric_Pad1.18x1.45mm_HandSolder, symbol Device:C
- added Cin2: 22u, Capacitor_SMD:C_0805_2012Metric_Pad1.18x1.45mm_HandSolder, symbol Device:C
- added D10: HB3, LED_SMD:LED_0805_2012Metric_Pad1.15x1.40mm_HandSolder, symbol Device:LED
- added D11: DB1, LED_SMD:LED_0805_2012Metric_Pad1.15x1.40mm_HandSolder, symbol Device:LED
- added D12: DB2, LED_SMD:LED_0805_2012Metric_Pad1.15x1.40mm_HandSolder, symbol Device:LED
- added D13: HB4, LED_SMD:LED_0805_2012Metric_Pad1.15x1.40mm_HandSolder, symbol Device:LED
- added D2: HB_CHG, LED_SMD:LED_0805_2012Metric_Pad1.15x1.40mm_HandSolder, symbol Device:LED
- added D8: HB1, LED_SMD:LED_0805_2012Metric_Pad1.15x1.40mm_HandSolder, symbol Device:LED
- added D9: HB2, LED_SMD:LED_0805_2012Metric_Pad1.15x1.40mm_HandSolder, symbol Device:LED
- added H1, H2, H3, H4: MountingHole, MountingHole:MountingHole_3.2mm_M3, symbol Mechanical:MountingHole
- added J1: ST-LINK Connector, Connector_IDC:IDC-Header_2x10_P2.54mm_Vertical, symbol Connector_Generic:Conn_02x10_Odd_Even
- added J8: USB4125-GF-A_REVA2, Downloaded_footprints:GCT_USB4125-GF-A_REVA2, symbol Downloaded_symbols:USB4125-GF-A_REVA2
- added J9: Extra GPIO Header, Connector_IDC:IDC-Header_2x05_P2.54mm_Vertical, symbol Connector_Generic:Conn_02x05_Odd_Even
- added L1: 1u, Inductor_SMD:L_1206_3216Metric_Pad1.42x1.75mm_HandSolder, symbol Device:L
- added L2: 1.3u, Inductor_SMD:L_1206_3216Metric_Pad1.42x1.75mm_HandSolder, symbol Device:L
- added R10: 10m, Resistor_SMD:R_0805_2012Metric_Pad1.20x1.40mm_HandSolder, symbol Device:R_US
- added R11, R12: 5.1k, Resistor_SMD:R_0805_2012Metric_Pad1.20x1.40mm_HandSolder, symbol Device:R_US
- added R58: 10k, Resistor_SMD:R_0805_2012Metric_Pad1.20x1.40mm_HandSolder, symbol Device:R_US
- added R59, R60: 100k, Resistor_SMD:R_0805_2012Metric_Pad1.20x1.40mm_HandSolder, symbol Device:R_US
- added R61, R62, R63, R64, R65, R66: 1k, Resistor_SMD:R_0805_2012Metric_Pad1.20x1.40mm_HandSolder, symbol Device:R_US
- added RIset1: 910, Resistor_SMD:R_0805_2012Metric_Pad1.20x1.40mm_HandSolder, symbol Device:R_US
- added Rchg1: 1.5k, Resistor_SMD:R_0805_2012Metric_Pad1.20x1.40mm_HandSolder, symbol Device:R_US
- added Rfbb1, Rfbb2: 137k, Resistor_SMD:R_0805_2012Metric_Pad1.20x1.40mm_HandSolder, symbol Device:R_US
- added Rfbt1, Rfbt2: 768k, Resistor_SMD:R_0805_2012Metric_Pad1.20x1.40mm_HandSolder, symbol Device:R_US
- added S1: PEC11R-4220F-S0024, Downloaded_footprints:XDCR_PEC11R-4220F-S0024, symbol Downloaded_symbols:PEC11R-4220F-S0024
- added SW1: SW_Push, Button_Switch_THT:SW_Tactile_Straight_KSA0Axx1LFTR, symbol Switch:SW_Push
- added TH1: Thermistor, Resistor_THT:R_Axial_DIN0204_L3.6mm_D1.6mm_P7.62mm_Horizontal, symbol Device:Thermistor
- added U1: STM32F767ZIT6, Downloaded_footprints:LQFP144-20x20mm_STM, symbol Downloaded_symbols:STM32F767ZIT6
- added U2, U6: TPS63020DSJR, Downloaded_footprints:TPS63020DSJR, symbol Downloaded_symbols:TPS63020DSJR
- added U3: MAX17055ETB+T, Downloaded_footprints:MAX17055, symbol Downloaded_symbols:MAX17055ETB+T
- added U4: 2.8_240x320_touch_sd_spi, Downloaded_footprints:2.8_tft_240x320_touch_sd_spi, symbol Downloaded_symbols:2.8_240x320_touch_sd_spi
- added U7: BQ21040DBVR, Downloaded_footprints:DBV0006A_N, symbol Downloaded_symbols:BQ21040DBVR
- BT1: footprint (none) -> Connector_Molex:Molex_CLIK-Mate_502386-0270_1x02-1MP_P1.25mm_Horizontal
Connections:
- net GND: now also C23.1, C24.2, C25.2, C26.2, C27.2, C28.2, C29.2, C30.2, C31.2, C32.2, C33.2, C34.2, C35.2, C36.2, C37.2, C38.2, C39.2, C4.2, C40.2, C41.2, C42.2, C43.2, C44.2, C45.2, C46.2, C47.2, C48.2, C49.2, C50.2, C6.2, C7.1, Cin1.2, Cin2.2, Cout2.2, Cout5.2, CvinA1.2, CvinA2.2, D10.1 (K), D11.1 (K), D12.1 (K), D13.1 (K), D8.1 (K), D9.1 (K), J1.10 (Pin_10), J1.12 (Pin_12), J1.14 (Pin_14), J1.16 (Pin_16), J1.18 (Pin_18), J1.20 (Pin_20), J1.4 (Pin_4), J1.6 (Pin_6), J1.8 (Pin_8), J8.A12 (GND), J8.B12 (GND__1), J8.S1 (SHIELD), J8.S2 (SHIELD__1), J8.S3 (SHIELD__2), J8.S4 (SHIELD__3), R10.2, R11.2, R12.2, R59.1, RIset1.2, Rfbb1.2, Rfbb2.2, S1.SH1 (SHIELD), S1.SH2 (SHIELD__1), SW1.1, TH1.2, U1.107 (VSS), U1.120 (VSS), U1.130 (VSS), U1.16 (VSS), U1.31 (VSSA), U1.38 (VSS), U1.51 (VSS), U1.61 (VSS), U1.83 (VSS), U1.94 (VSS), U2.13 (PS/SYNC), U2.2 (GND), U3.5 (CSN), U4.2 (GND), U6.13 (PS/SYNC), U6.2 (GND), U7.5 (VSS)
- net V_Batt+: now reaches BT1.1 (+)
- net V_Batt+: now also C4.1, C7.2, Cin2.1, Cin3.1, R66.2, Rchg1.1, U2.10 (VIN), U3.10 (BATT), U6.10 (VIN), U7.2 (OUT)
- net V_Batt-: now reaches BT1.2 (-)
- net V_Batt-: now also C5.2, R10.1, U3.6 (CSP)
- new net: D10.2 (A), R63.1
- new net: D8.2 (A), R61.2
- new net: R64.1, U1.114 (PD0)
- new net: D11.2 (A), R64.2
- new net: C5.1, U3.7 (REG)
- new net: C23.2, C24.1, U1.106 (VCAP_2), U1.71 (VCAP_1)
- new net: Cout3.2, Cout4.1
- new net: Cout4.2, Cout5.1
- new net: Cin1.1, Cin3.2
- new net: Cout1.1, Cout6.2
- new net: CvinA2.1, U6.1 (VINA), U6.12 (EN)
- new net: Rfbb2.1, Rfbt2.2, U6.3 (FB)
- new net: L1.1, U6.6 (L2)
- new net: L1.2, U6.8 (L1)
- new net: R58.2, S1.1
- new net: J8.A5 (CC1), R11.1
- new net: D2.2 (A), Rchg1.2
- new net: RIset1.1, U7.4 (ISET)
- new net: D9.2 (A), R62.1
- new net: R65.1, U1.115 (PD1)
- new net: D12.2 (A), R65.2
- new net: J8.B5 (CC2), R12.1
- new net: L2.1, U2.6 (L2)
- new net: L2.2, U2.8 (L1)
- new net: TH1.1, U7.1 (TS)
- new net: Cout1.2, Cout2.1
- new net: CvinA1.1, U2.1 (VINA), U2.12 (EN)
- new net: D2.1 (K), U7.3 (CHG_N)
- new net: D13.2 (A), R66.1
- new net: Rfbb1.1, Rfbt1.2, U2.3 (FB)
- new net 3.3V_0.5A: Cout3.1, R62.2, Rfbt1.1, U2.4 (VOUT)
- new net 3.3V_0.6A: C25.1, C26.1, C27.1, C28.1, C29.1, C30.1, C31.1, C32.1, C33.1, C34.1, C35.1, C36.1, C37.1, C38.1, C39.1, C40.1, C41.1, C42.1, C43.1, C44.1, C45.1, C46.1, C47.1, C48.1, C49.1, Cout6.1, R58.1, R60.1, R61.1, Rfbt2.1, S1.C (COM), U1.108 (VDD), U1.131 (VDD), U1.144 (VDD), U1.17 (VDD), U1.30 (VDD), U1.32 (VREF+), U1.33 (VDDA), U1.39 (VDD), U1.52 (VDD), U1.6 (VBAT), U1.62 (VDD), U1.72 (VDD), U1.84 (VDD), U4.1 (VCC), U4.8 (LED), U6.4 (VOUT)
- new net 5V_In: C6.1, J8.A9 (VBUS), R63.2, U7.6 (IN)
- new net Batt_ALRT: U1.29 (PC3), U3.8 (ALRT)
- new net Batt_SCL: U1.44 (PC4), U3.3 (SCL)
- new net Batt_SDA: U1.45 (PC5), U3.4 (SDA)
- new net ENC_CLK: S1.A, U1.42 (PA6)
- new net ENC_DT: S1.B, U1.97 (PC7)
- new net ENC_SW: R59.2, S1.2, U1.43 (PA7)
- new net LCD_CLK: U1.41 (PA5), U4.7 (SCK)
- new net LCD_CS: U1.136 (PB6), U4.3 (CS)
- new net LCD_D/C: U1.27 (PC1), U4.5 (D/C)
- new net LCD_MISO: U1.139 (PB8), U4.9 (SDO(MISO))
- new net LCD_MOSI: U1.137 (PB7), U4.6 (SDI(MOSI))
- new net LCD_RST: U1.140 (PB9), U4.4 (RESET)
- new net NRST: C50.1, J1.15 (Pin_15), R60.2, SW1.2, U1.25 (NRST)
- new net PE0: J9.1 (Pin_1), U1.141 (PE0)
- new net PE1: J9.2 (Pin_2), U1.142 (PE1)
- new net PE2: J9.3 (Pin_3), U1.1 (PE2)
- new net PE3: J9.4 (Pin_4), U1.2 (PE3)
- new net PE4: J9.5 (Pin_5), U1.3 (PE4)
- new net PE5: J9.6 (Pin_6), U1.4 (PE5)
- new net PE6: J9.7 (Pin_7), U1.5 (PE6)
- new net PE7: J9.8 (Pin_8), U1.58 (PE7)
- new net PE8: J9.9 (Pin_9), U1.59 (PE8)
- new net PE9: J9.10 (Pin_10), U1.60 (PE9)
- new net SWCLK: J1.9 (Pin_9), U1.109 (PA14)
- new net SWDIO: J1.7 (Pin_7), U1.105 (PA13)
- new net SWO: J1.13 (Pin_13), U1.133 (PB3)
- new net TDI: J1.5 (Pin_5), U1.110 (PA15)
- new net TRST: J1.3 (Pin_3), U1.134 (PB4)
- new net micPin1: U1.37 (PA3)
- new net micPin2: U1.26 (PC0)
- new net micPin3: U1.28 (PC2)
- new net micPin4: U1.13 (PF3)
- new net micPin5: U1.15 (PF5)
- new net micPin6: U1.22 (PF10)
- new net motorPin1: U1.124 (PG9)
- new net motorPin2: U1.129 (PG14)
- new net motorPin3: U1.66 (PE13)
- new net motorPin4: U1.85 (PD14)
- new net motorPin5: U1.54 (PF14)
- new net motorPin6: U1.64 (PE11)
- no-connect marks 0 -> 107
Other:
- note added: "3.3 V @ 0.5 A Buck/Boost"
- note added: "3.3 V @ 0.6 A Buck/Boost"
- note added: "910 = 600 mA charge current"
- note added: "BMS"
- note added: "CHECK EPAD"
- note added: "CHECK EPAD & THERM"
- note added: "Debug GPIO"
- note added: "Debug LEDs"
- note added: "LCD"
- note added: "MCU Block(s)"
- note added: "MCU Reset Circuit"
- note added: "Mounting Holes"
- note added: "Rotary Encoder"
- note added: "ST-LINK"
- note added: "USB-C Charging Circuit"
- note removed: "+4.5"
- moved on the sheet: BT1

Commit message: Added updated schematic
Includes BOM, new footprints
Parts:
- removed BT1: Battery_Cell, Connector_Molex:Molex_CLIK-Mate_502386-0270_1x02-1MP_P1.25mm_Horizontal, symbol Device:Battery_Cell
- removed C25, C27, C28, C29, C30, C31, C32, C33, C34, C35, C36, C37, C38, C39, C40, C42, C43, C44, C45, C46, C47, C48, CvinA1, CvinA2: 100n, Capacitor_SMD:C_0805_2012Metric_Pad1.18x1.45mm_HandSolder, symbol Device:C
- removed C26, C49: 1u, Capacitor_SMD:C_0805_2012Metric_Pad1.18x1.45mm_HandSolder, symbol Device:C
- removed C41: 4.7u, Capacitor_SMD:C_0805_2012Metric_Pad1.18x1.45mm_HandSolder, symbol Device:C
- removed Cin3, Cout3, Cout4, Cout5, Cout6: 10u, Capacitor_SMD:C_0805_2012Metric_Pad1.18x1.45mm_HandSolder, symbol Device:C
- removed D8: HB1, LED_SMD:LED_0805_2012Metric_Pad1.15x1.40mm_HandSolder, symbol Device:LED
- removed D9: HB2, LED_SMD:LED_0805_2012Metric_Pad1.15x1.40mm_HandSolder, symbol Device:LED
- removed J1: ST-LINK Connector, Connector_IDC:IDC-Header_2x10_P2.54mm_Vertical, symbol Connector_Generic:Conn_02x10_Odd_Even
- removed R61, R62: 1k, Resistor_SMD:R_0805_2012Metric_Pad1.20x1.40mm_HandSolder, symbol Device:R_US
- removed Rfbb1, Rfbb2: 137k, Resistor_SMD:R_0805_2012Metric_Pad1.20x1.40mm_HandSolder, symbol Device:R_US
- removed Rfbt1, Rfbt2: 768k, Resistor_SMD:R_0805_2012Metric_Pad1.20x1.40mm_HandSolder, symbol Device:R_US
- removed U2, U6: TPS63020DSJR, Downloaded_footprints:TPS63020DSJR, symbol Downloaded_symbols:TPS63020DSJR
- added C1, C10, C12, C13, C14, C16, C2, C3, C4, C5, C6, C8, C9: 100n, Capacitor_SMD:C_0805_2012Metric_Pad1.18x1.45mm_HandSolder, symbol Device:C
- added C11, C18, C7: 1u, Capacitor_SMD:C_0805_2012Metric_Pad1.18x1.45mm_HandSolder, symbol Device:C
- added C15: 4.7u, Capacitor_SMD:C_0805_2012Metric_Pad1.18x1.45mm_HandSolder, symbol Device:C
- added D1, D17, D2, D4, D5, D6, D7, D8, D9: ESD, Downloaded_footprints:DIO_RSB5.6SM_ROM, symbol Diode:1N47xxA
- added D3: ESD, Downloaded_footprints:DIODE_CDSOD323-T05C_BRN, symbol Diode:1N47xxA
- added DHB1, DHB2: LED, LED_SMD:LED_0805_2012Metric_Pad1.15x1.40mm_HandSolder, symbol Device:LED
- added E1: HZ0805E601R-10, Downloaded_footprints:FB_HZ0805E601R-10, symbol Downloaded_symbols:HZ0805E601R-10
- added J1: Mic-Motor connector, Downloaded_footprints:CONN10_302-S101_OST, symbol Connector_Generic:Conn_02x05_Odd_Even
- added J2: ST-LINK Connector, Downloaded_footprints:CONN10_302-S101_OST, symbol Connector_Generic:Conn_02x05_Odd_Even
- added J5: S2B-XH-A, Downloaded_footprints:JST_S2B-XH-A, symbol Downloaded_symbols:S2B-XH-A
- added R10, R13, R14, R28, R3, R4, R5, R7, R8, R9: 220, Resistor_SMD:R_0805_2012Metric_Pad1.20x1.40mm_HandSolder, symbol Device:R_US
- added R11, R12: 1k, Resistor_SMD:R_0805_2012Metric_Pad1.20x1.40mm_HandSolder, symbol Device:R_US
- added U3, U4: TPS63001DRCR, Downloaded_footprints:TPS63001DRCR, symbol Downloaded_symbols:TPS63001DRCR
- Cin1: footprint Capacitor_SMD:C_0805_2012Metric_Pad1.18x1.45mm_HandSolder -> Downloaded_footprints:CAP_MSAS21-9_TAY
- Cin2: value 22u -> 10u; footprint Capacitor_SMD:C_0805_2012Metric_Pad1.18x1.45mm_HandSolder -> Downloaded_footprints:CAP_MSAS21-9_TAY
- Cout1, Cout2: value 10u -> 47u; footprint Capacitor_SMD:C_0805_2012Metric_Pad1.18x1.45mm_HandSolder -> Downloaded_footprints:CAP_2012_TDK
- DDB1: renamed from D11; value DB1 -> LED
- DDB2: renamed from D12; value DB2 -> LED
- DHB3: renamed from D13; value HB4 -> LED
- DHB4: renamed from D10; value HB3 -> LED
- L1: value 1u -> 1.5u; footprint Inductor_SMD:L_1206_3216Metric_Pad1.42x1.75mm_HandSolder -> Downloaded_footprints:INDC2520X100N
- L2: value 1.3u -> 1.5u; footprint Inductor_SMD:L_1206_3216Metric_Pad1.42x1.75mm_HandSolder -> Downloaded_footprints:INDC2520X100N
- SW1: footprint Button_Switch_THT:SW_Tactile_Straight_KSA0Axx1LFTR -> Downloaded_footprints:SW_D6R90_F2_LFS
- TH1: footprint Resistor_THT:R_Axial_DIN0204_L3.6mm_D1.6mm_P7.62mm_Horizontal -> Downloaded_footprints:THRMC2012X130N
- renumbered C24 to C17, C23 to C19, C5 to C20, C4 to C21, C50 to C22, C6 to C23, C7 to C24, D2 to D10, H4 to H2, H2 to H3, H3 to H4, J8 to J3, J9 to J4, R64 to R1, R66 to R15, R58 to R16, R63 to R17, R12 to R18, R60 to R19, R65 to R2, R59 to R20, R11 to R21, R10 to R6, U3 to U2, U7 to U5, U4 to U6
Connections:
- net 5V_In is gone; now on an unnamed net: C23.1, J3.A9 (VBUS), R17.2, U5.6 (IN)
- net V_Batt- is gone; now on net GND: C20.2, R6.1, U2.6 (CSP)
- net GND: now also Cout1.2, U2.11 (EPAD), C1.2, C10.2, C11.2, C12.2, C13.2, C14.2, C15.2, C16.2, C18.2, C2.2, C3.2, C4.2, C5.2, C6.2, C7.2, C8.2, C9.2, D1.2 (A), D17.2 (A), D2.2 (A), D3.2 (A), D4.2 (A), D5.2 (A), D6.2 (A), D7.2 (A), D8.2 (A), D9.2 (A), DHB1.1 (K), DHB2.1 (K), J1.10 (Pin_10), J2.3 (Pin_3), J2.4 (Pin_4), J5.2, U3.11 (PAD), U3.3 (PGND), U3.9 (GND), U4.11 (PAD), U4.3 (PGND), U4.9 (GND)
- net NRST: now also D17.1 (K), J2.1 (Pin_1), R28.2; no longer C22.1, R19.2, SW1.2
- net PE1: now also J4.1 (Pin_1); no longer J4.2 (Pin_2)
- net PE2: now also J4.2 (Pin_2); no longer J4.3 (Pin_3)
- net PE3: now also J4.3 (Pin_3); no longer J4.4 (Pin_4)
- net PE4: now also J4.4 (Pin_4); no longer J4.5 (Pin_5)
- net PE5: now also J4.5 (Pin_5); no longer J4.6 (Pin_6)
- net PE6: now also J4.6 (Pin_6); no longer J4.7 (Pin_7)
- net PE7: now also J4.7 (Pin_7); no longer J4.8 (Pin_8)
- net PE8: now also J4.8 (Pin_8); no longer J4.9 (Pin_9)
- net PE9: now also J4.9 (Pin_9); no longer J4.10 (Pin_10)
- net SWCLK: now also J2.6 (Pin_6)
- net SWDIO: now also J2.2 (Pin_2)
- net V_Batt+: now also Cin1.1, J5.1, U3.5 (VIN), U3.6 (EN), U3.7 (PS_SYNC), U3.8 (VINA), U4.5 (VIN), U4.6 (EN), U4.7 (PS_SYNC), U4.8 (VINA)
- net micPin1: now also D4.1 (K), R7.1
- net micPin2: now also D1.1 (K), R3.1
- net micPin3: now also D6.1 (K), R9.1
- net micPin4: now also D9.1 (K), R14.1
- net motorPin1: now also D2.1 (K), R4.1
- net motorPin2: now also D5.1 (K), R8.1
- net motorPin3: now also D8.1 (K), R13.1
- net motorPin4: now also D7.1 (K), R10.1
- net 3.3V_0.42A: now reaches Cout1.1
- net 3.3V_0.42A: now also Cout2.1, R16.1, R19.1, S1.C (COM), U1.108 (VDD), U1.121 (VDDSDMMC), U1.131 (VDD), U1.144 (VDD), U1.17 (VDD), U1.30 (VDD), U1.39 (VDD), U1.52 (VDD), U1.6 (VBAT), U1.62 (VDD), U1.72 (VDD), U1.84 (VDD), U1.95 (VDDUSB), U6.1 (VCC), U6.8 (LED), C1.1, C10.1, C11.1, C12.1, C13.1, C14.1, C15.1, C2.1, C3.1, C4.1, C5.1, C6.1, C7.1, C8.1, C9.1, D3.1 (K), E1.1, R11.1, R12.1, R5.1, U3.1 (VOUT), U3.10 (FB), U4.1 (VOUT), U4.10 (FB)
- net at L1.1: now also U3.4 (L1)
- net at L1.2: now also U3.2 (L2)
- net at L2.1: now also U4.4 (L1)
- net at L2.2: now also U4.2 (L2)
- net PE10: now reaches U1.63 (PE10)
- net PE10: now also J4.10 (Pin_10)
- removed net 3.3V_0.6A: R16.1, R19.1, S1.C (COM), U1.108 (VDD), U1.131 (VDD), U1.144 (VDD), U1.17 (VDD), U1.30 (VDD), U1.32 (VREF+), U1.33 (VDDA), U1.39 (VDD), U1.52 (VDD), U1.6 (VBAT), U1.62 (VDD), U1.72 (VDD), U1.84 (VDD), U6.1 (VCC), U6.8 (LED)
- net PE0: no longer names the net of U1.141 (PE0)
- net PE0: no longer J4.1 (Pin_1)
- net TRST: no longer names the net of U1.134 (PB4)
- net micPin5: no longer names the net of U1.15 (PF5)
- net micPin6: no longer names the net of U1.22 (PF10)
- net motorPin5: no longer names the net of U1.54 (PF14)
- net motorPin6: no longer names the net of U1.64 (PE11)
- new net: J1.9 (Pin_9), R5.2
- new net: DHB1.2 (A), R11.2
- new net: DHB2.2 (A), R12.2
- new net: J1.7 (Pin_7), R8.2
- new net: J1.3 (Pin_3), R4.2
- new net: C22.1, R19.2, R28.1, SW1.2
- new net: J1.1 (Pin_1), R7.2
- new net: J1.6 (Pin_6), R14.2
- new net: J1.5 (Pin_5), R3.2
- new net: J1.2 (Pin_2), R9.2
- new net: J1.8 (Pin_8), R10.2
- new net: J1.4 (Pin_4), R13.2
- new net 3V3A: C16.1, C18.1, E1.2, U1.32 (VREF+), U1.33 (VDDA)
- no-connect marks 107 -> 90
Other:
- note added: "Battery"
- note added: "Buck-Boost 3.3V @ 0.42A"
- note added: "Buck-Boost 3.3V @ 0.5A"
- note added: "Mic-Motor Connector w/ESD"
- note removed: "3.3 V @ 0.5 A Buck/Boost"
- note removed: "3.3 V @ 0.6 A Buck/Boost"
- note removed: "CHECK EPAD"
- note removed: "CHECK EPAD & THERM"
- moved on the sheet: C17, C19, C20, C21, C22, R19, R6, SW1, U1B, U2
